File: xt60PDU.kicad_sch (KiCad schematic)
At the start: 7 parts, among them J1 Conn_01x02_Pin, J2 Conn_01x02_Socket, J3 Conn_01x02_Socket, J4 Conn_01x02_Socket, J5 Conn_01x02_Socket

Commit message: Replace the 1812 PTC footprint with one that is shorted by default
Parts:
- F2: footprint Fuse:Fuse_1812_4532Metric -> SMD:SolderJumper-2_1812_Bridged_3.2mm
Changed lines of the file:
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@@
 			)
 		)
-		(property "Footprint" "Fuse:Fuse_1812_4532Metric"
+		(property "Footprint" "SMD:SolderJumper-2_1812_Bridged_3.2mm"
 			(at 46.99 21.59 0)
 			(effects

Commit message: Add v1.0 with fixed pin numbering and connector orientation
Connections:
- net GND: now also J1.2 (Pin_2); no longer J1.1 (Pin_1)
- net VBAT: now also J1.1 (Pin_1); no longer J1.2 (Pin_2)
Other:
- moved on the sheet: J1
Changed lines of the file:
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@@
 	(generator_version "9.0")
 	(paper "A4")
-	(text_box "NOTE: angled footprint have GND on pin 1, vertical ones have VCC on PIN1"
-		(exclude_from_sim no)
-		(at 25.146 32.512 0)
-		(size 39.624 5.588)
-		(margins 0.9525 0.9525 0.9525 0.9525)
-		(stroke
-			(width 0)
-			(type solid)
-		)
-		(fill
-			(type none)
-		)
-		(effects
-			(font
-				(size 1.27 1.27)
-			)
-			(justify left top)
-		)
-	)
 	(junction
 		(at 66.04 22.86)
@@
 	)
 	(label "VBAT"
-		(at 25.4 25.4 180)
+		(at 25.4 22.86 180)
 		(effects
 			(font
@@
 	(symbol
 		(lib_id "Connector:Conn_01x02_Pin")
-		(at 30.48 27.94 180)
+		(at 20.32 25.4 0)
 		(unit 1)
 		(exclude_from_sim no)
@@
 		(dnp no)
 		(property "Reference" "J1"
-			(at 28.956 26.67 0)
+			(at 21.844 26.67 0)
 			(effects
 				(font
@@
 		)
 		(property "Value" "Conn_01x02_Pin"
-			(at 29.845 30.48 0)
+			(at 20.955 22.86 0)
 			(effects
 				(font
@@
 		)
 		(property "Footprint" "Connector_AMASS:AMASS_XT60PW-M_1x02_P7.20mm_Horizontal"
-			(at 30.48 27.94 0)
+			(at 20.32 25.4 0)
 			(effects
 				(font
@@
 		)
 		(property "Datasheet" "~"
-			(at 30.48 27.94 0)
+			(at 20.32 25.4 0)
 			(effects
 				(font
@@
 		)
 		(property "Description" "Generic connector, single row, 01x02, script generated"
-			(at 30.48 27.94 0)
-			(effects
-				(font
+			(at 20.32 25.4 0)
+			(effects
+				(font
